File: Miasma_IO_smd/Miasma_IO_smd.kicad_pcb (KiCad board)
At the start: 2 copper layers, 99.1 x 99.1 mm, 137 parts, among them P1 CONN_01X12, P2 CONN_01X10, P3 CONN_01X10, P4 CONN_01X12, P5 Conn_01x02, P6 Conn_01x02, P7 CONN_01X01, Q1 MMBT3904, Q2 MMBT3904, Q3 MMBT3904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

Commit message: Improve silkscreen of Miasma I/O board, fix kicad symbols
Silkscreen had only a few minor legibility issues.

Replace some symbols now unavailable in the Kicad 10 library.
Kicad project has been saved as a Kicad 10 project now.

Exported iBOM.

Signed-off-by: Nicholas Marrone <nickmarrone@gmail.com>
Other:
- net class Default removed
